File: PCB/Sliphub.kicad_sch (KiCad schematic)
At the start: 20 parts, among them J1 USB_C_Receptacle_USB2.0_16P, J2 USB_C_Receptacle_USB2.0_16P, J3 USB_C_Receptacle_USB2.0_16P, J4 USB_A, J5 USB_A, U1 SL2.1A

Commit message: add BOM for JLCPCB for PCBA
Parts:
- D1: LCSC C154551 -> C8678
Changed lines of the file:
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@@
 			)
 		)
-		(property "LCSC" "C154551"
+		(property "LCSC" "C8678"
 			(at 50.8 38.1 90)
 			(effects
